File: Simple_8088/Simple_8088.sch (KiCad schematic (older format))
At the start: 19 parts, among them J1 Conn_02x22_Counter_Clockwise, SW1 RESET, U1 8088, U2 74LS257, U3 74LS573, U4 74LS245, U5 74LS04, U6 62256, U7 28C256, X1 OSC

Commit message: Changing RAM
Parts:
- removed U6: 62256, Package_DIP:DIP-28_W15.24mm, symbol Memory_RAM:CY62256-70PC
- removed U7: 28C256, Package_DIP:DIP-28_W15.24mm, symbol Memory_EEPROM:28C256
- added C10, C9: 0.1uF, Capacitor_THT:C_Disc_D4.3mm_W1.9mm_P5.00mm, symbol pspice:CAP
- added U6: AS6C4008, Package_DIP:DIP-32_W15.24mm, symbol Memory_RAM:AS6C4008-55PCN
- added U7: 27C512, Socket:DIP_Socket-28_W11.9_W12.7_W15.24_W17.78_W18.5_3M_228-1277-00-0602J, symbol Memory_EPROM:27C512
- added U8: 74LS573, Package_DIP:DIP-20_W7.62mm, symbol 74xx:74LS573
- added U9: 74LS138, Package_DIP:DIP-16_W7.62mm, symbol 74xx:74LS138
Connections:
- net A15_ is gone; now on net RESET_: U5.2
- net 5+: now also C10.2, C9.2, U6.32 (VCC), U7.28 (VCC), U8.20 (VCC), U9.16 (VCC)
- net A0: now also U6.12 (A0), U7.10 (A0); no longer J1.12 (Pin_12)
- net A1: now also U6.11 (A1), U7.9 (A1); no longer J1.11 (Pin_11)
- net A10: now also U6.23 (A10), U7.21 (A10)
- net A11: now also U6.25 (A11), U7.23 (A11)
- net A12: now also U6.4 (A12), U7.2 (A12)
- net A13: now also U6.28 (A13), U7.26 (A13)
- net A14: now also U6.3 (A14), U7.27 (A14)
- net A15: now also U6.31 (A15), U7.1 (A15); no longer U5.1
- net A2: now also U6.10 (A2), U7.8 (A2); no longer J1.10 (Pin_10)
- net A3: now also U6.9 (A3), U7.7 (A3); no longer J1.9 (Pin_9)
- net A4: now also U6.8 (A4), U7.6 (A4); no longer J1.8 (Pin_8)
- net A5: now also U6.7 (A5), U7.5 (A5); no longer J1.7 (Pin_7)
- net A6: now also U6.6 (A6), U7.4 (A6); no longer J1.6 (Pin_6)
- net A7: now also U6.5 (A7), U7.3 (A7); no longer J1.5 (Pin_5)
- net A8: now also U6.27 (A8), U7.25 (A8)
- net A9: now also U6.26 (A9), U7.24 (A9)
- net ALE: now also U8.11 (Load)
- net D0: now also U6.13 (DQ0), U7.11 (D0); no longer J1.20 (Pin_20)
- net D1: now also U6.14 (DQ1), U7.12 (D1); no longer J1.19 (Pin_19)
- net D2: now also U6.15 (DQ2), U7.13 (D2); no longer J1.18 (Pin_18)
- net D3: now also U6.17 (DQ3), U7.15 (D3); no longer J1.17 (Pin_17)
- net D4: now also U6.18 (DQ4), U7.16 (D4); no longer J1.16 (Pin_16)
- net D5: now also U6.19 (DQ5), U7.17 (D5); no longer J1.15 (Pin_15)
- net D6: now also U6.20 (DQ6), U7.18 (D6); no longer J1.14 (Pin_14)
- net D7: now also U6.21 (DQ7), U7.19 (D7); no longer J1.13 (Pin_13)
- net GND: now also C10.1, C9.1, U6.16 (VSS), U7.14 (GND), U8.10 (GND), U9.4 (E1), U9.5 (E2), U9.8 (GND); no longer U1.18 (INTR)
- net HOLDA: now also U8.1 (OE)
- net IORD: no longer J1.3 (Pin_3)
- net IOWR: no longer J1.4 (Pin_4)
- net MRD: now also U6.24 (OE#), U7.20 (~CE)
- net MWR: now also U6.29 (WE#)
- net RESET: now also U5.1; no longer U5.3
- net RESET_: no longer U5.4
- net A19_: now reaches U1.35 (A19/S6)
- net A19_: now also U8.5 (D3), U8.9 (D7)
- net A18_: now reaches U1.36 (A18/S5)
- net A18_: now also U8.8 (D6)
- net A17_: now reaches U1.37 (A17/S4)
- net A17_: now also U8.7 (D5)
- net A16_: now reaches U1.38 (A16/S3)
- net A16_: now also U8.6 (D4)
- new net 512K_CS: U6.22 (CE#), U8.16 (Q3)
- new net A16: U6.2 (A16), U8.15 (Q4), U9.1 (A0)
- new net A17: U6.30 (A17), U8.14 (Q5), U9.2 (A1)
- new net A18: U6.1 (A18), U8.13 (Q6), U9.3 (A2)
- new net A19: U8.12 (Q7), U9.6 (E3)
- new net INTR: U1.18 (INTR)
- new net ROM_CS: U7.22 (~OE), U9.7 (O7)
Changed lines of the file:
@@
-$EndComp
-$Comp
-L Memory_EEPROM:28C256 U7
-U 1 1 66171932
-P 8525 4225
-F 0 "U7" H 8525 5506 50  0000 C CNN
-F 1 "28C256" H 8525 5415 50  0000 C CNN
-F 2 "Package_DIP:DIP-28_W15.24mm" H 8525 4225 50  0001 C CNN
-F 3 "http://ww1.microchip.com/downloads/en/DeviceDoc/doc0006.pdf" H 8525 4225 50  0001 C CNN
-	1    8525 4225
-	1    0    0    -1
-$EndComp
-$Comp
-L Memory_RAM:CY62256-70PC U6
-U 1 1 66173257
-P 6850 4100
-F 0 "U6" H 6850 5181 50  0000 C CNN
-F 1 "62256" H 6850 5090 50  0000 C CNN
-F 2 "Package_DIP:DIP-28_W15.24mm" H 6850 4000 50  0001 C CNN
-F 3 "https://ecee.colorado.edu/~mcclurel/Cypress_SRAM_CY62256.pdf" H 6850 4000 50  0001 C CNN
-	1    6850 4100
-	1    0    0    -1
 $EndComp
 $Comp
@@
 GND
 Text Label 1950 2250 2    50   ~ 0
-GND
+INTR
 Text Label 1950 2850 2    50   ~ 0
 GND
@@
 Text Label 1150 6350 2    50   ~ 0
 RESET
-Text Label 7400 1950 2    50   ~ 0
+Text Label 7400 1375 2    50   ~ 0
 RESET
-Text Label 8000 1950 0    50   ~ 0
+Text Label 8000 1375 0    50   ~ 0
 RESET_
-Text Label 8000 1375 0    50   ~ 0
-A15_
-Text Label 7400 1375 2    50   ~ 0
-A15
 Text Label 8575 1350 0    50   ~ 0
 5+
@@
 Text Label 8525 5325 0    50   ~ 0
 GND
-Text Label 6850 5000 0    50   ~ 0
+Text Label 6850 5400 0    50   ~ 0
 GND
 Text Label 6350 3400 2    50   ~ 0
@@
 Text Label 7350 4600 0    50   ~ 0
 MWR
-Text Label 8125 4925 2    50   ~ 0
-MWR
-Text Label 8125 5125 2    50   ~ 0
-A15_
-Text Label 7350 4300 0    50   ~ 0
+Text Label 8125 4825 2    50   ~ 0
+A15
+Text Label 6350 4900 2    50   ~ 0
 A15
 $Comp
@@
 	1    0    0    -1
 $EndComp
-Text Label 10375 4450 2    50   ~ 0
-D7
-Text Label 10375 4550 2    50   ~ 0
-D6
-Text Label 10375 4650 2    50   ~ 0
-D5
-Text Label 10375 4750 2    50   ~ 0
-D4
-Text Label 10375 4850 2    50   ~ 0
-D3
-Text Label 10375 4950 2    50   ~ 0
-D2
-Text Label 10375 5050 2    50   ~ 0
-D1
-Text Label 10375 5150 2    50   ~ 0
-D0
-Text Label 10375 4350 2    50   ~ 0
-A0
-Text Label 10375 4250 2    50   ~ 0
-A1
-Text Label 10375 4150 2    50   ~ 0
-A2
-Text Label 10375 4050 2    50   ~ 0
-A3
-Text Label 10375 3950 2    50   ~ 0
-A4
-Text Label 10375 3850 2    50   ~ 0
-A5
-Text Label 10375 3750 2    50   ~ 0
-A6
-Text Label 10375 3650 2    50   ~ 0
-A7
 Text Label 10875 4350 0    50   ~ 0
 A0
@@
 Text Label 10875 3450 0    50   ~ 0
 IORD
-Text Label 10375 3550 2    50   ~ 0
-IOWR
-Text Label 10375 3450 2    50   ~ 0
-IORD
 Text Label 10375 5250 2    50   ~ 0
 GND
@@
 Text Label 700  6175 2    50   ~ 0
 GND
+$Comp
+L 74xx:74LS573 U8
+U 1 1 662E9544
+P 6250 1675
+F 0 "U8" H 6250 2656 50  0000 C CNN
+F 1 "74LS573" H 6250 2565 50  0000 C CNN
+F 2 "Package_DIP:DIP-20_W7.62mm" H 6250 1675 50  0001 C CNN
+F 3 "74xx/74hc573.pdf" H 6250 1675 50  0001 C CNN
+	1    6250 1675
+	1    0    0    -1
+$EndComp
+Text Label 3350 3650 0    50   ~ 0
+A16_
+Text Label 3350 3750 0    50   ~ 0
+A17_
+Text Label 3350 3850 0    50   ~ 0
+A18_
+Text Label 3350 3950 0    50   ~ 0
+A19_
+Text Label 5750 1575 2    50   ~ 0
+A16_
+Text Label 5750 1675 2    50   ~ 0
+A17_
+Text Label 5750 1775 2    50   ~ 0
+A18_
+Text Label 5750 1875 2    50   ~ 0
+A19_
+Text Label 6750 1575 0    50   ~ 0
+A16
+Text Label 6750 1675 0    50   ~ 0
+A17
+Text Label 6750 1775 0    50   ~ 0
+A18
+Text Label 6750 1875 0    50   ~ 0
+A19
+Text Label 6250 875  0    50   ~ 0
+5+
+Text Label 6250 2475 0    50   ~ 0
+GND
+$Comp
+L pspice:CAP C9
+U 1 1 662ED8DD
+P 6575 650
+F 0 "C9" V 6260 650 50  0000 C CNN
+F 1 "0.1uF" V 6351 650 50  0000 C CNN
+F 2 "Capacitor_THT:C_Disc_D4.3mm_W1.9mm_P5.00mm" H 6575 650 50  0001 C CNN
+F 3 "~" H 6575 650 50  0001 C CNN
+	1    6575 650
+	0    1    1    0
+$EndComp
+Text Label 6325 650  2    50   ~ 0
+5+
+Text Label 6825 650  0    50   ~ 0
+GND
+$Comp
+L Memory_RAM:AS6C4008-55PCN U6
+U 1 1 662EE794
+P 6850 4300
+F 0 "U6" H 6850 5581 50  0000 C CNN
+F 1 "AS6C4008" H 6850 5490 50  0000 C CNN
+F 2 "Package_DIP:DIP-32_W15.24mm" H 6850 4400 50  0001 C CNN
+F 3 "https://www.alliancememory.com/wp-content/uploads/pdf/AS6C4008.pdf" H 6850 4400 50  0001 C CNN
+	1    6850 4300
+	1    0    0    -1
+$EndComp
+Text Label 6350 5000 2    50   ~ 0
+A16
+Text Label 6350 5100 2    50   ~ 0
+A17
+Text Label 6350 5200 2    50   ~ 0
+A18
+Text Label 5750 2175 2    50   ~ 0
+HOLDA
+Text Label 5750 2075 2    50   ~ 0
+ALE
+Text Label 7350 4400 0    50   ~ 0
+512K_CS
+$Comp
+L Memory_EPROM:27C512 U7
+U 1 1 662FA8F9
+P 8525 4225
+F 0 "U7" H 8525 5506 50  0000 C CNN
+F 1 "27C512" H 8525 5415 50  0000 C CNN
+F 2 "Socket:DIP_Socket-28_W11.9_W12.7_W15.24_W17.78_W18.5_3M_228-1277-00-0602J" H 8525 4225 50  0001 C CNN
+F 3 "http://ww1.microchip.com/downloads/en/DeviceDoc/doc0015.pdf" H 8525 4225 50  0001 C CNN
+	1    8525 4225
+	1    0    0    -1
+$EndComp
+Text Label 8125 5125 2    50   ~ 0
+ROM_CS
+$Comp
+L 74xx:74LS138 U9
+U 1 1 66300322
+P 10300 1875
+F 0 "U9" H 10300 2656 50  0000 C CNN
+F 1 "74LS138" H 10300 2565 50  0000 C CNN
+F 2 "Package_DIP:DIP-16_W7.62mm" H 10300 1875 50  0001 C CNN
+F 3 "http://www.ti.com/lit/gpn/sn74LS138" H 10300 1875 50  0001 C CNN
+	1    10300 1875
+	1    0    0    -1
+$EndComp
+$Comp
+L pspice:CAP C10
+U 1 1 6630150C
+P 10650 875
+F 0 "C10" V 10335 875 50  0000 C CNN
+F 1 "0.1uF" V 10426 875 50  0000 C CNN
+F 2 "Capacitor_THT:C_Disc_D4.3mm_W1.9mm_P5.00mm" H 10650 875 50  0001 C CNN
+F 3 "~" H 10650 875 50  0001 C CNN
+	1    10650 875
+	0    1    1    0
+$EndComp
+Text Label 10400 875  2    50   ~ 0
+5+
+Text Label 10900 875  0    50   ~ 0
+GND
+Text Label 9800 1575 2    50   ~ 0
+A16
+Text Label 9800 1775 2    50   ~ 0
+A18
+Text Label 9800 1675 2    50   ~ 0
+A17
+Text Label 9800 2175 2    50   ~ 0
+GND
+Text Label 9800 2075 2    50   ~ 0
+A19
+Text Label 9800 2275 2    50   ~ 0
+GND
+Text Label 10300 2575 2    50   ~ 0
+GND
+Text Label 10300 1275 2    50   ~ 0
+5+
+Text Label 10800 2275 0    50   ~ 0
+ROM_CS
+Text Label 5750 1475 2    50   ~ 0
+A19_
+Text Label 6750 1475 0    50   ~ 0
+512K_CS
 $EndSCHEMATC
